File: Hardware/kicad/mini.kicad_sch (KiCad schematic)
At the start: 29 parts, among them J1 JS40F-I, J10 MOTOR-I, J11 MOTOR-D, J13 XT30PW-M, J2 JS40F-LI, J3 QRE-I, J4 JS40F-M, J5 QRE-M, J6 JS40F-D, J7 JS40F-LD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

Commit message: actu 29/05
Parts:
- added H1, H2, H3, H4: Mounting_Hole, EESTN5:hole_3mm, symbol EESTN5:Mounting_Hole
- added LED2, LED4: Rojo, EESTN5:Led_0805, symbol EESTN5:LED
- added LED3, LED5: Verde, EESTN5:Led_0805, symbol EESTN5:LED
- added R5, R6, R7, R8: 22k, EESTN5:R_0805, symbol EESTN5:R
Connections:
- net GND: now also LED2.2 (K), LED3.2 (K), LED4.2 (K), LED5.2 (K)
- net JS40F-LD: now also U3.6 (GPIO6); no longer U3.5 (GPIO5)
- net MI_A: now also U3.10 (GPIO10); no longer U3.1 (GPIO1)
- net QRE-D: now also U3.5 (GPIO5); no longer U3.6 (GPIO6)
- net QRE-I: now also U3.1 (GPIO1); no longer U3.10 (GPIO10)
- net at J11.1, U4.7 (BO1), U4.8 (BO2): now also R7.1
- net at J11.2, U4.5 (FO1), U4.6 (FO2): now also R8.1
- net at J10.2, U2.5 (FO1), U2.6 (FO2): now also R6.1
- net at J10.1, U2.7 (BO1), U2.8 (BO2): now also R5.1
- new net: LED4.1 (A), R7.2
- new net: LED3.1 (A), R6.2
- new net: LED2.1 (A), R5.2
- new net: LED5.1 (A), R8.2
Other:
- moved on the sheet: C5, C6, J1, J10, J11, J2, J3, J4, J5, J6, J7, J8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
